File: Eurorack/LFO_VC/LFO_VC.kicad_pcb (KiCad board)
At the start: 2 copper layers, 114 x 88 mm, 105 parts, among them J1 CV1, J10 CFV, J11 FFV, J12 PWC, J13 PW90, J14 PW10, J16 PWXV, J17 PWR, J2 CV2, J3 CV3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

Commit message: Update LFO_VC with fab outputs
Parts:
- removed R62: 27K, Resistor_THT:R_Axial_DIN0207_L6.3mm_D2.5mm_P7.62mm_Horizontal
- removed R63: 4.7M, Resistor_THT:R_Axial_DIN0207_L6.3mm_D2.5mm_P7.62mm_Horizontal
- added G***: LOGO, LOGO, F.Cu at (142.5, 62.6)
- added G***: LOGO, LOGO, F.Cu at (98.5, 63.0)
- C12: value 10pF -> 10p
- J8: value RMP -> RAMP
- LED1: value LED1 -> ~; footprint Connector_Wire:SolderWire-0.127sqmm_1x01_D0.48mm_OD1mm_Custom -> Connector_Wire:SolderWire-0.5sqmm_1x01_D0.9mm_OD2.1mm
- Q1, Q2, Q3, Q4, Q5, Q6: footprint Package_TO_SOT_THT:TO-92_Inline -> Package_TO_SOT_THT:TO-92_Inline_Wide
- R45: value 9.1K -> 6.1K
- VR46: value 2K -> 5K
- moved R60 15.2 mm to (165.5, 93.7)
- moved Q6 14.9 mm to (164.0, 86.1)
- moved REF** 8.00 mm to (165.2, 139.8)
- moved REF** 8.00 mm to (165.2, 63.8)
- moved J6 7.02 mm to (156.8, 138.1), turned to 180 degrees
- moved Q4 6.95 mm to (86.3, 127.0), turned to 180 degrees
- moved Q5 6.92 mm to (86.3, 135.4), turned to 180 degrees
- moved R3 6.46 mm to (99.6, 88.4)
- moved J4 6.25 mm to (153.2, 83.5)
- moved C6 5.86 mm to (160.5, 133.8)
- moved R39 5.84 mm to (81.2, 109.5)
- moved LED1 5.53 mm to (164.0, 82.8)
- moved R38 5.49 mm to (150.9, 79.1)
- moved R15 5.44 mm to (154.0, 79.1)
- moved R61 4.85 mm to (162.7, 98.1)
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Connections:
- net /C_INV_SQR renamed /INV_SQR
- net Net-(J4-T) renamed /TRI
- net Net-(J5-T) renamed /SIN
- net Net-(J6-T) renamed /SQR
- net Net-(J7-T) renamed /SAW
- net Net-(J8-T) renamed /RMP
- Q4 pad 1: Net-(Q4-G) -> Net-(Q4-D)
- Q4 pad 3: Net-(Q4-D) -> Net-(Q4-G)
- Q5 pad 1: Net-(Q5-G) -> Net-(Q5-D)
- Q5 pad 3: Net-(Q5-D) -> Net-(Q5-G)
Routing:
- net GND: track 339.2 -> 52.2 mm, vias 3 -> 2
- net /INV_SQR: track 119.5 -> 105.8 mm
- net Net-(LED1-A): track 14.0 -> 3.30 mm
- net +12V: track 377.1 -> 366.8 mm, vias 3 -> 0
- net Net-(U6A--): track 53.7 -> 45.6 mm
- net Net-(Q4-S): track 160.0 -> 152.1 mm
- net /SQR: track 12.8 -> 19.6 mm
- net Net-(Q1-E): track 20.9 -> 14.2 mm
- net Net-(R45-Pad2): track 15.7 -> 10.1 mm
- net Net-(Q4-D): track 11.9 -> 6.95 mm
- net Net-(Q5-S): track 194.1 -> 189.2 mm
- net Net-(Q4-G): track 5.30 -> 9.89 mm
- net Net-(Q6-B): track 6.72 -> 11.2 mm
- net Net-(U2A--): track 28.9 -> 24.7 mm
- net CV_OUTPUT: track 24.1 -> 19.9 mm, vias 1 -> 0
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- added copper zone on B.Cu, net GND
- added copper zone on F.Cu, net GND
Other:
- board size 114 x 88 mm -> 100.8 x 84.8 mm
- board text added: "Based on design by Ray Wilson of MFOS"
- board text added: "github.com/mitchreyno"
- board text removed: "Design by Ray Wilson of MFOS"
