File: Eurorack/LFO_VC/LFO_VC.kicad_sch (KiCad schematic)
At the start: 106 parts, among them J1 ${SIM.PARAMS}, J10 CFV, J11 FFV, J12 PWC, J13 PW90, J14 PW10, J16 ${SIM.PARAMS}, J17 PWR, J2 ${SIM.PARAMS}, J3 ${SIM.PARAMS}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

Commit message: Update LFO_VC with fab outputs
Parts:
- LED1: footprint SolderWire-0.127sqmm_1x01_D0.48mm_OD1mm_Custom -> Connector_Wire:SolderWire-0.5sqmm_1x01_D0.9mm_OD2.1mm
- V1, V2: now left out of the parts list
Other:
- moved on the sheet: R23
