File: Eurorack/Clocky/Clocky.kicad_sch (KiCad schematic)
At the start: 2 parts, among them U2 74HC165

Commit message: Update finalised clocky files
Parts:
- removed U2: 74HC165, Package_DIP:DIP-16_W7.62mm_Socket_LongPads, symbol 74xx:74HC165
- added C1: 10uF, symbol Device:C_Polarized
- added C6: 100nF, symbol Device:C
- added J1: IDC_02x08, Connector_IDC:IDC-Header_2x08_P2.54mm_Vertical, symbol Connector_Generic:Conn_02x05_Odd_Even
- added J10: G, Connector_Audio:Jack_3.5mm_QingPu_WQP-PJ398SM_Vertical_CircularHoles, symbol Connector_Audio:AudioJack2_SwitchT
- added J11: H, Connector_Audio:Jack_3.5mm_QingPu_WQP-PJ398SM_Vertical_CircularHoles, symbol Connector_Audio:AudioJack2_SwitchT
- added J2: TRG, Connector_Audio:Jack_3.5mm_QingPu_WQP-PJ398SM_Vertical_CircularHoles, symbol Connector_Audio:AudioJack2_SwitchT
- added J3: RST, Connector_Audio:Jack_3.5mm_QingPu_WQP-PJ398SM_Vertical_CircularHoles, symbol Connector_Audio:AudioJack2_SwitchT
- added J4: A, Connector_Audio:Jack_3.5mm_QingPu_WQP-PJ398SM_Vertical_CircularHoles, symbol Connector_Audio:AudioJack2_SwitchT
- added J5: B, Connector_Audio:Jack_3.5mm_QingPu_WQP-PJ398SM_Vertical_CircularHoles, symbol Connector_Audio:AudioJack2_SwitchT
- added J6: C, Connector_Audio:Jack_3.5mm_QingPu_WQP-PJ398SM_Vertical_CircularHoles, symbol Connector_Audio:AudioJack2_SwitchT
- added J7: D, Connector_Audio:Jack_3.5mm_QingPu_WQP-PJ398SM_Vertical_CircularHoles, symbol Connector_Audio:AudioJack2_SwitchT
- added J8: E, Connector_Audio:Jack_3.5mm_QingPu_WQP-PJ398SM_Vertical_CircularHoles, symbol Connector_Audio:AudioJack2_SwitchT
- added J9: F, Connector_Audio:Jack_3.5mm_QingPu_WQP-PJ398SM_Vertical_CircularHoles, symbol Connector_Audio:AudioJack2_SwitchT
- added Q14, Q15, Q16, Q17, Q18, Q19, Q20, Q21, Q22, Q23: 2N3904, Package_TO_SOT_THT:TO-92_Inline_Wide, symbol Transistor_BJT:2N3904
- added R37, R38: 100K, symbol Device:R
- added R39, R40, R41, R42, R43, R44, R45, R46, R47, R48, R49, R50, R51, R52, R53, R54, R55, R56: 10K, symbol Device:R
Connections:
- net +5V: now also R39.1, R40.1
- net GND: now also C1.2, C6.1, J1.3 (Pin_3), J1.4 (Pin_4), J1.5 (Pin_5), J1.6 (Pin_6), J1.7 (Pin_7), J1.8 (Pin_8), J10.S, J11.S, J2.S, J3.S, J4.S, J5.S, J6.S, J7.S, J8.S, J9.S, Q14.1 (E), Q15.1 (E), Q16.1 (E), Q17.1 (E), Q18.1 (E), Q19.1 (E), Q20.1 (E), Q21.1 (E), Q22.1 (E), Q23.1 (E)
- net LED_Mux/LED_MUX_CLK: now reaches A1.10 (D7)
- net LED_Mux/LED_MUX_RST: now reaches A1.11 (D8)
- net Switches_SR/SR_PL_IN: now reaches A1.12 (D9)
- net Switches_SR/SR_CLK: now reaches A1.13 (D10)
- net Switches_SR/SR_SER_OUT: now reaches A1.14 (D11)
- net OUT_G: now reaches A1.15 (D12)
- net OUT_G: now also R51.1
- net OUT_H: now reaches A1.16 (D13)
- net OUT_H: now also R52.1
- net OUT_A: now reaches A1.19 (A0)
- net OUT_A: now also R41.1
- net OUT_B: now reaches A1.20 (A1)
- net OUT_B: now also R43.1
- net OUT_C: now reaches A1.21 (A2)
- net OUT_C: now also R45.1
- net OUT_F: now reaches A1.24 (A5)
- net OUT_F: now also R50.1
- net +12V: now reaches A1.30 (VIN)
- net +12V: now also C1.1, C6.2, J1.10 (Pin_10), J1.9 (Pin_9), R42.2, R44.2, R46.2, R48.2, R53.2, R54.2, R55.2, R56.2
- net at A1.5 (D2): now also Q14.3 (C), R39.2
- net at A1.6 (D3): now also Q15.3 (C), R40.2
- net LED_Mux/LED_R: now reaches A1.7 (D4)
- net LED_Mux/LED_G: now reaches A1.8 (D5)
- net LED_Mux/LED_B: now reaches A1.9 (D6)
- net LED_Mux/LED_CLK renamed OUT_D
- net OUT_D: now also R47.1
- net LED_Mux/LED_RESET renamed OUT_E
- net OUT_E: now also R49.1
- new net: Q21.2 (B), R50.2
- new net: J9.T, Q21.3 (C), R54.1
- new net: Q22.2 (B), R51.2
- new net: J10.T, Q22.3 (C), R55.1
- new net: J4.T, Q16.3 (C), R42.1
- new net: Q18.2 (B), R45.2
- new net: J5.T, Q17.3 (C), R44.1
- new net: Q23.2 (B), R52.2
- new net: J11.T, Q23.3 (C), R56.1
- new net: J8.T, Q20.3 (C), R53.1
- new net: Q16.2 (B), R41.2
- new net: J7.T, Q19.3 (C), R48.1
- new net: Q14.2 (B), R37.2
- new net: Q17.2 (B), R43.2
- new net: J6.T, Q18.3 (C), R46.1
- new net: J3.T, R38.1
- new net: J2.T, R37.1
- new net: Q19.2 (B), R47.2
- new net: Q15.2 (B), R38.2
- new net: Q20.2 (B), R49.2
Other:
- added sheet Switches_SR (Clocky_Switches_SR.kicad_sch)
- sheet LED_Mux ports: added LED_B, LED_G, LED_MUX_CLK, LED_MUX_RST, LED_R; removed LED_CH_B, LED_CH_G, LED_CH_R, LED_CLK, LED_RESET
- moved on the sheet: A1
