File: Eurorack/Clocky/Clocky_LED_Mux.kicad_sch (KiCad schematic)
At the start: 51 parts, among them Q1 2N3904, Q10 2N3904, Q11 2N3904, Q12 2N3904, Q13 2N3904, Q2 2N3904, Q3 2N3904, Q4 2N3904, Q5 2N3904, Q6 2N3904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

Commit message: Update finalised clocky files
Parts:
- added C4: 100nF, symbol Device:C
- R23: value 10K -> 330R
- R24, R26: value 10K -> 470R
Connections:
- net +5V: now also C4.1
- net GND: now also C4.2
- net LED_CH_B renamed LED_B
- net LED_CH_G renamed LED_G
- net LED_CH_R renamed LED_R
- net LED_CLK renamed LED_MUX_CLK
- net LED_RESET renamed LED_MUX_RST
Other:
- moved on the sheet: R1
